File: hardware/schematic/mainboard.sch (EAGLE design)
At the start: 34 parts, among them Q1 8MHz, Q2 32.768KHz, U1 PIC32MX460F512L TQFP100

Commit message: Cleaned up schematic and added power supply to it
Parts:
- removed R1: 10K, SparkFun-Passives:RESISTOR0402-RES
- removed R10, R12, R17, R2, R3, R5: 4.7K, SparkFun-Passives:RESISTOR0402-RES
- added B1: DF01S, lizardworx:DF01S
- added C1: (no value), rcl:CPOL-USE10-20
- added C2: 1uF, SparkFun-Passives:CAP0402-CAP
- added J1: POWER_JACKPTH, lizardworx:POWER_JACKPTH
- added OK1: MOC3032S, lizardworx:MOC3032S
- added PWR: BLUE, SparkFun:LED0603
- added R13, R15, R28: (no value), SparkFun-Passives:RESISTOR0603-RES
- added R14: 10K, SparkFun-Passives:RESISTOR0603-RES
- added R22, R23, R24, R25, R26, R27: 4.7K, SparkFun-Passives:RESISTOR0603-RES
- added U2: RECOM_X.X_REG78XX, lizardworx:RECOM_X.X_REG78XX
- R4, R6, R7, R8, R9: device SparkFun:RESISTOR0402 -> SparkFun-Passives:RESISTOR0603-RES
Connections:
- new net N$1: B1.AC1, J1.PWR
- new net N$2: B1.AC2, J1.GND, J1.GNDBREAK
- new net N$3: B1.+, C1.+, U2.IN
- new net N$4: PWR.A, R15.1
- net 3.3V: now also C2.1, R14.1, R15.2, R22.2, R23.2, R24.2, R25.1, R26.2, R9.1, U2.OUT; no longer R1.1, R10.2, R12.2, R17.2, R2.1, R3.2, R9.2
- net GND: now also B1.-, C1.-, C2.2, PWR.C, R27.1, U2.GND; no longer R5.1
- net N$5: now also R25.2; no longer R2.2
- net SD_CS: now also R14.2; no longer R1.2
- net USBID: now also R9.2; no longer R9.1
- net WF_CK: now also R23.1; no longer R12.1
- net WF_DI: now also R22.1; no longer R10.1
- net WF_INT: now also R24.1; no longer R17.1
- net WF_RESET: now also R26.1; no longer R3.1
- net WF_WP: now also R27.2; no longer R5.2
Other:
- note added: "RTC Crystal"
- note removed: "PIC32MX795F512L can be substituted"
- moved on the sheet: C10, C11, C16, C17, C6, C7, C8, C9, J5, LED1, LED2, LED3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

Commit message: Finished full system schematic
Parts:
- removed J5: (no value), SchmalzHaus:M08
- removed R9: 10K, SparkFun-Passives:RESISTOR0603-RES
- added JP1: (no value), SparkFun-Connectors:M05LOCK
- added OK10, OK11, OK12, OK13, OK14, OK15, OK16, OK2, OK3, OK4, OK5, OK6, OK7, OK8, OK9: MOC3032S, lizardworx:MOC3032S
- added R1, R10, R12, R17, R19, R21, R3, R30, R32, R34, R36, R38, R40, R42, R44: 33, SparkFun-Passives:RESISTOR0603-RES
- added R11, R16, R18, R2, R20, R29, R31, R33, R35, R37, R39, R41, R43, R45, R5: 330, SparkFun-Passives:RESISTOR0603-RES
- added R46, R47, R48, R49, R50: 4.7K, SparkFun-Passives:RESISTOR0603-RES
- added T1, T10, T11, T12, T13, T14, T15, T16, T2, T3, T4, T5, T6, T7, T8, T9: LF-TRIACSOT223, lizardworx:LF-TRIACSOT223
- added U$21: USB-MINIB-5PIN, SparkFun-Connectors:USB-MINIB-5PIN
- added U$22: M40, SparkFun-Connectors:M40
- C1: value (none) -> 3300uF
- R13: value (none) -> 33
- R14: value 10K -> 4.7K
- R28: value (none) -> 330
Connections:
- net N$2 renamed AC_NEUTRAL
- new net AC_HOT: B1.AC1, J1.PWR, R1.1, R10.1, R12.1, R13.1, R17.1, R19.1, R21.1, R3.1, R30.1, R32.1, R34.1, R36.1, R38.1, R40.1, R42.1, R44.1, T1.A2, T10.A2, T11.A2, T12.A2, T13.A2, T14.A2, T15.A2, T16.A2, T2.A2, T3.A2, T4.A2, T5.A2, T6.A2, T7.A2, T8.A2, T9.A2
- new net CNTRL_1: R2.2
- new net CNTRL_10: R11.2
- new net CNTRL_11: R16.2
- new net CNTRL_12: R18.2
- new net CNTRL_13: R35.2
- new net CNTRL_14: R37.2
- new net CNTRL_15: R39.2
- new net CNTRL_16: R41.2
- new net CNTRL_2: R28.2
- new net CNTRL_3: R29.2
- new net CNTRL_4: R20.2
- new net CNTRL_5: R33.2
- new net CNTRL_6: R31.2
- new net CNTRL_7: R45.2
- new net CNTRL_8: R43.2
- new net CNTRL_9: R5.2
- new net N$10: R14.1, R46.1
- new net N$11: R47.2, R48.2
- new net N$12: OK2.A2, R1.2
- new net N$13: OK9.A1, T9.G
- new net N$14: OK2.A1, T2.G
- new net N$15: R49.2, R50.1
- new net N$17: OK3.A, R5.1
- new net N$18: OK3.A2, R3.2
- new net N$2: OK1.A, R28.1
- new net N$21: OK3.A1, T3.G
- new net N$26: OK4.A, R11.1
- new net N$27: OK4.A2, R10.2
- new net N$28: OK10.A, R33.1
- new net N$29: OK4.A1, T4.G
- new net N$32: OK5.A, R16.1
- new net N$33: OK5.A2, R12.2
- new net N$34: OK10.A2, R32.2
- new net N$36: OK5.A1, T5.G
- new net N$39: OK6.A, R18.1
- new net N$40: OK6.A2, R17.2
- new net N$41: OK10.A1, T10.G
- new net N$42: OK6.A1, T6.G
- new net N$45: OK7.A, R20.1
- new net N$46: OK7.A2, R19.2
- new net N$48: OK7.A1, T7.G
- new net N$51: OK8.A, R29.1
- new net N$52: OK8.A2, R21.2
- new net N$53: OK11.A, R35.1
- new net N$54: OK8.A1, T8.G
- new net N$57: OK11.A2, R34.2
- new net N$58: OK11.A1, T11.G
- new net N$6: OK1.A2, R13.2
- new net N$61: OK12.A, R37.1
- new net N$62: OK12.A2, R36.2
- new net N$63: OK12.A1, T12.G
- new net N$66: OK13.A, R39.1
- new net N$67: OK13.A2, R38.2
- new net N$68: OK13.A1, T13.G
- new net N$7: OK9.A2, R30.2
- new net N$71: OK14.A, R41.1
- new net N$72: OK14.A2, R40.2
- new net N$73: OK14.A1, T14.G
- new net N$76: OK15.A, R43.1
- new net N$77: OK15.A2, R42.2
- new net N$78: OK15.A1, T15.G
- new net N$8: OK1.A1, T1.G
- new net N$81: OK16.A, R45.1
- new net N$82: OK16.A2, R44.2
- new net N$83: OK16.A1, T16.G
- new net N$9: OK2.A, R2.1
- new net STATION_1: T2.A1
- new net STATION_10: T4.A1
- new net STATION_11: T5.A1
- new net STATION_12: T6.A1
- new net STATION_13: T11.A1
- new net STATION_14: T12.A1
- new net STATION_15: T13.A1
- new net STATION_16: T14.A1
- new net STATION_2: T1.A1
- new net STATION_3: T8.A1
- new net STATION_4: T7.A1
- new net STATION_5: T10.A1
- new net STATION_6: T9.A1
- new net STATION_7: T16.A1
- new net STATION_8: T15.A1
- new net STATION_9: T3.A1
- net 3.3V: now also JP1.2, R46.2, R48.1, R50.2; no longer J5.2, R14.1, R9.1
- net D+: now also U$21.D+
- net D-: now also U$21.D-
- net GND: now also JP1.3, OK1.C, OK10.C, OK11.C, OK12.C, OK13.C, OK14.C, OK15.C, OK16.C, OK2.C, OK3.C, OK4.C, OK5.C, OK6.C, OK7.C, OK8.C, OK9.C, U$21.GND, U$21.MTN1, U$21.MTN2, U$21.MTN3, U$21.MTN4; no longer J5.3
- net N$1: now also OK9.A, R31.1; no longer B1.AC1, J1.PWR
- net PGC: now also JP1.5; no longer J5.5
- net PGD: now also JP1.4; no longer J5.4
- net RB0: no longer J5.8
- net RB1: no longer J5.7
- net RB2: no longer J5.6
- net USBID: now also R49.1, U$21.ID; no longer R9.2
- net VBUS: now also U$21.VBUS
- net VPP: now also JP1.1, R47.1; no longer J5.1
Other:
- note added: "Kevin Sidwar"
- note added: "v1.0"
- moved on the sheet: B1, C1, C10, C11, C14, C15, C16, C17, C2, C4, C5, C6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

Commit message: Clean up schematic - no electrical changes
Parts:
- removed C17: 11pf, SparkFun:CAP0402
- removed R50: 4.7K, SparkFun-Passives:RESISTOR0603-RES
- added C3: 0.1uF, SparkFun:CAP0402
- added R9: 4.7K, SparkFun-Passives:RESISTOR0603-RES
- C10: value 0.1uF -> 10uF; device SparkFun02-20-08:CAP0402 -> SparkFun02-20-08:CAP_POL3528
- C11: value 0.1uF -> 18pF
- C14: value 18pF -> 11pf
- C5: value 10uF -> 0.1uF; device SparkFun02-20-08:CAP_POL3528 -> SparkFun:CAP0402
- C7: device SparkFun:CAP0402 -> SparkFun02-20-08:CAP0402
- R1, R12, R13, R19, R21, R30, R32: value 33 -> 330
- R10, R17, R3: value 33 -> 4.7K
- R11, R16, R2, R4, R5, R6, R7, R8: value 330 -> 4.7K
- R14, R22, R23, R24, R25, R26, R27: value 4.7K -> 330
- R15: value (none) -> 330
- R35, R37, R39, R41, R43, R45: value 330 -> 33
- R46, R47, R48, R49: value 4.7K -> 33
- renumbered C15 to C12, C16 to C13
Connections:
- net 3.3V: now also C3.1, C4.1, C5.1, R1.2, R10.2, R11.2, R12.2, R13.2, R14.2, R17.2, R3.2, R5.1, R8.1, R9.2; no longer C10.1, C11.1, C9.1, R22.2, R23.2, R24.2, R25.1, R26.2, R4.2, R46.2, R48.1, R50.2, R6.2, R8.2
- net AC_HOT: now also R35.1, R37.1, R39.1, R41.1, R43.1, R45.1, R46.1, R47.1, R48.1, R49.1; no longer R1.1, R10.1, R12.1, R13.1, R17.1, R19.1, R21.1, R3.1, R30.1, R32.1
- net CNTRL_1: now also R18.2; no longer R2.2
- net CNTRL_10: now also R27.2; no longer R11.2
- net CNTRL_11: now also R28.2; no longer R16.2
- net CNTRL_12: now also R29.2; no longer R18.2
- net CNTRL_13: now also R30.2; no longer R35.2
- net CNTRL_14: now also R31.2; no longer R37.2
- net CNTRL_15: now also R32.2; no longer R39.2
- net CNTRL_16: now also R33.2; no longer R41.2
- net CNTRL_2: now also R19.2; no longer R28.2
- net CNTRL_3: now also R20.2; no longer R29.2
- net CNTRL_4: now also R21.2; no longer R20.2
- net CNTRL_5: now also R22.2; no longer R33.2
- net CNTRL_6: now also R23.2; no longer R31.2
- net CNTRL_7: now also R24.2; no longer R45.2
- net CNTRL_8: now also R25.2; no longer R43.2
- net CNTRL_9: now also R26.2; no longer R5.2
- net GND: now also C10.-, C11.1, C14.2, C3.2, C5.2, R6.1; no longer C10.2, C11.2, C14.1, C17.2, C5.-, R27.1
- net N$1: now also R23.1; no longer R31.1
- net N$10: now also R16.1, R17.1; no longer R14.1, R46.1
- net N$11: now also R4.2, R5.2; no longer R47.2, R48.2
- net N$110: now also C10.+, C9.1; no longer C4.1, C5.+
- net N$12: now also R34.2; no longer R1.2
- net N$15: now also R2.2, R3.1; no longer R49.2, R50.1
- net N$17: now also R26.1; no longer R5.1
- net N$18: now also R42.2; no longer R3.2
- net N$2: now also R19.1; no longer R28.1
- net N$20: now also R15.1; no longer R8.1
- net N$22: now also R14.1; no longer R7.1
- net N$23: now also R13.1; no longer R6.1
- net N$26: now also R27.1; no longer R11.1
- net N$27: now also R43.2; no longer R10.2
- net N$28: now also R22.1; no longer R33.1
- net N$32: now also R28.1; no longer R16.1
- net N$33: now also R44.2; no longer R12.2
- net N$34: now also R38.2; no longer R32.2
- net N$35: now also R12.1; no longer R4.1
- net N$39: now also R29.1; no longer R18.1
- net N$4: now also R1.1; no longer R15.1
- net N$40: now also R45.2; no longer R17.2
- net N$45: now also R21.1; no longer R20.1
- net N$46: now also R37.2; no longer R19.2
- net N$5: now also R8.2; no longer R25.2
- net N$51: now also R20.1; no longer R29.1
- net N$52: now also R36.2; no longer R21.2
- net N$53: now also R30.1; no longer R35.1
- net N$57: now also R46.2; no longer R34.2
- net N$6: now also R35.2; no longer R13.2
- net N$61: now also R31.1; no longer R37.1
- net N$62: now also R47.2; no longer R36.2
- net N$66: now also R32.1; no longer R39.1
- net N$67: now also R48.2; no longer R38.2
- net N$7: now also R39.2; no longer R30.2
- net N$71: now also R33.1; no longer R41.1
- net N$72: now also R49.2; no longer R40.2
- net N$76: now also R25.1; no longer R43.1
- net N$77: now also R41.2; no longer R42.2
- net N$81: now also R24.1; no longer R45.1
- net N$82: now also R40.2; no longer R44.2
- net N$9: now also R18.1; no longer R2.1
- net OSC1: now also C11.2; no longer C14.2
- net RC13: now also C14.1; no longer C17.1
- net SD_CS: now also R16.2; no longer R14.2
- net USBID: now also R2.1; no longer R49.1
- net VPP: now also R4.1; no longer R47.1
- net WF_CK: now also R10.1; no longer R23.1
- net WF_DI: now also R9.1; no longer R22.1
- net WF_INT: now also R11.1; no longer R24.1
- net WF_RESET: now also R7.1; no longer R26.1
- net WF_WP: now also R6.2; no longer R27.2
Other:
- moved on the sheet: C11, C14, C4, C6, C7, C8, C9, R1, R10, R11, R12, R13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
