File: hardware/schematic/Power Supply.brd (EAGLE design)
At the start: 36.8 x 44.5 mm, 16 parts, among them J1 POWER_JACKPTH, U2 RECOM_X.X_REG78XX

Commit message: Increase trace widths on Power board.  Start motherboard layout
Parts:
- removed JP2, JP3: (no value), SparkFun-Connectors:1X02_LOCK_LONGPADS
- added F1: 500mA PTC Fuse, resistor:M1206
- C2: value (none) -> 1uF
- moved JP4 10.2 mm to (34.3, 14.0), turned to 270 degrees
Connections:
- new net N$1: C2.1, F1.2, U2.VOUT
- net 3.3V: now also F1.1; no longer C2.1, JP1.2, U2.VOUT
- net AC_HOT: no longer JP4.2
- net AC_NEUTRAL: now also JP4.2; no longer JP3.1, JP3.2
- net GND: now also JP1.2; no longer JP2.1, JP2.2
Routing:
- net 3.3V: track 27.8 -> 12.5 mm
- net N$1: track 0.00 -> 12.2 mm
- net AC_HOT: track 32.7 -> 24.0 mm
- net AC_NEUTRAL: track 32.2 -> 25.8 mm
- net GND: track 75.8 -> 73.9 mm
Other:
- board text added: "NEUT"
- board text added: "PTC"
- board text removed: "NEUTRAL"
