File: hardware/schematic/Valve Board.sch (EAGLE design)
At the start: 111 parts, among them J1 POWER_JACKPTH, Q1 8MHz, Q2 32.768KHz, T1 LF-TRIACSOT223, T10 LF-TRIACSOT223, T11 LF-TRIACSOT223, T12 LF-TRIACSOT223, T13 LF-TRIACSOT223, T14 LF-TRIACSOT223, T15 LF-TRIACSOT223, T16 LF-TRIACSOT223, T2 LF-TRIACSOT223, T3 LF-TRIACSOT223, T4 LF-TRIACSOT223, T5 LF-TRIACSOT223, T6 LF-TRIACSOT223, T7 LF-TRIACSOT223, T8 LF-TRIACSOT223, T9 LF-TRIACSOT223, U1 PIC32MX460F512L TQFP100, U2 RECOM_X.X_REG78XX

Commit message: Increase trace widths on Power board.  Start motherboard layout
Parts:
- removed B1: DF01S, lizardworx:DF01S
- removed C1: 3300uF, rcl:CPOL-USE10-20
- removed C10: 10uF, SparkFun02-20-08:CAP_POL3528
- removed C11, C12: 18pF, SparkFun:CAP0402
- removed C13, C14: 11pf, SparkFun:CAP0402
- removed C2: 1uF, SparkFun-Passives:CAP0402-CAP
- removed C3, C4, C5, C6, C8, C9: 0.1uF, SparkFun:CAP0402
- removed C7: 0.1uF, SparkFun02-20-08:CAP0402
- removed J1: POWER_JACKPTH, lizardworx:POWER_JACKPTH
- removed JP1: (no value), SparkFun-Connectors:M05LOCK
- removed LED1: WHITE, SparkFun:LED0603
- removed LED2: RED, SparkFun:LED0603
- removed LED3: YELLOW, SparkFun:LED0603
- removed PWR: BLUE, SparkFun:LED0603
- removed Q1: 8MHz, SparkFun11_03_09:CRYSTAL5X3
- removed Q2: 32.768KHz, SchmalzHaus:CRYSTAL32-SMD
- removed R1, R12, R13, R14, R15: 330, SparkFun-Passives:RESISTOR0603-RES
- removed R10, R11, R16, R17, R2, R3, R4, R5, R6, R7, R8, R9: 4.7K, SparkFun-Passives:RESISTOR0603-RES
- removed U$1: MRF24WB0MA, lizardworx:MRF24WB0MA
- removed U$21: USB-MINIB-5PIN, SparkFun-Connectors:USB-MINIB-5PIN
- removed U$22: M40, SparkFun-Connectors:M40
- removed U$3: SD_CARD_SOCKETSD, SparkFun-Connectors:SD_CARD_SOCKETSD
- removed U1: PIC32MX460F512L TQFP100, SchmalzHaus:PIC32MX4XXLTQFP100
- removed U2: RECOM_X.X_REG78XX, lizardworx:RECOM_X.X_REG78XX
- removed USB: GREEN, SparkFun:LED0603
Connections:
- removed net 3.3V: C2.1, C3.1, C4.1, C5.1, C6.1, C7.1, C8.1, JP1.2, R1.2, R10.2, R11.2, R12.2, R13.2, R14.2, R15.2, R17.2, R3.2, R5.1, R7.2, R8.1, R9.2, U$1.VDD@17, U$1.VDD@29, U$3.VCC, U1.AVDD, U1.ENVREG, U1.VDD1, U1.VDD2, U1.VDD3, U1.VDD4, U1.VDD5, U1.VUSB, U2.OUT
- removed net AC_NEUTRAL: B1.AC2, J1.GND, J1.GNDBREAK
- removed net D+: U$21.D+, U1.D+/RG2
- removed net D-: U$21.D-, U1.D-/RG3
- removed net N$10: R16.1, R17.1
- removed net N$11: R4.2, R5.2
- removed net N$110: C10.+, C9.1, U1.VCAP/VDDCORE
- removed net N$15: R2.2, R3.1
- removed net N$20: R15.1, USB.A
- removed net N$22: LED1.A, R14.1
- removed net N$23: LED2.A, R13.1
- removed net N$3: B1.+, C1.+, U2.IN
- removed net N$35: LED3.A, R12.1
- removed net N$4: PWR.A, R1.1
- removed net N$5: R8.2, U$1.JTAG_TCK
- removed net OSC1: C11.2, Q1.1, U1.OSC1/CLKI/RC12
- removed net OSC2: C12.2, Q1.2, U1.OSC2/CLKO/RC15
- removed net PGC: JP1.5, U1.PGC2/EMUC2/AN6/OCFA/RB6
- removed net PGD: JP1.4, U1.PGD2/EMUD2/AN7/RB7
- removed net RA0: U1.TMS/RA0
- removed net RA1: U1.TCK/RA1
- removed net RA10: U1.PMA6/VREF+/CVREF+/RA10
- removed net RA14: U1.SCL1/INT3/RA14
- removed net RA15: U1.SDA1/INT4/RA15
- removed net RA2: U1.SCL2/RA2
- removed net RA4: U1.TDI/RA4
- removed net RA5: U1.TDO/RA5
- removed net RA6: U1.TRCLK/RA6
- removed net RA7: U1.TRD3/RA7
- removed net RA9: U1.PMA7/VREF-/CVREF-/RA9
- removed net RB0: U1.PGD1/EMUD1/AN0/CN2/RB0
- removed net RB1: U1.PGC1/EMUC1/AN1/CN3/RB1
- removed net RB10: U1.CVREFOUT/PMA13/AN10/RB10
- removed net RB11: U1.PMA12/AN11/RB11
- removed net RB12: U1.PMA11/AN12/RB12
- removed net RB13: U1.PMA10/AN13/RB13
- removed net RB14: U1.PMALH/PMA1/AN14/RB14
- removed net RB15: U1.PMALL/PMA0/AN15/OCFB/CN12/RB15
- removed net RB2: U1.C2IN-/AN2/CN4/RB2
- removed net RB3: U1.C2IN+/AN3/CN5/RB3
- removed net RB4: U1.C1IN-/AN4/CN6/RB4
- removed net RB5: U1.VBUSON/C1IN+/AN5/CN7/RB5
- removed net RB8: U1.C1OUT/AN8/RB8
- removed net RB9: U1.C2OUT/AN9/RB9
- removed net RC1: U1.T2CK/RC1
- removed net RC13: C14.1, Q2.1, U1.SOSCI/CN1/RC13
- removed net RC14: C13.1, Q2.2, U1.SOSCO/T1CK/CN0/RC14
- removed net RC2: U1.T3CK/RC2
- removed net RC3: U1.T4CK/RC3
- removed net RD1: U1.OC2/RD1
- removed net RD11: U1.IC4/PMCS1/PMA14/RD11
- removed net RD12: U1.PMD12/IC5/RD12
- removed net RD13: U1.PMD13/CN19/RD13
- removed net RD14: U1.CN20/U1CTS/RD14
- removed net RD15: U1.U1RTS/BCLK1/CN21/RD15
- removed net RD2: U1.OC3/RD2
- removed net RD3: U1.OC4/RD3
- removed net RD4: U1.PMWR/OC5/CN13/RD4
- removed net RD5: U1.PMRD/CN14/RD5
- removed net RD6: U1.PMD14/CN15/RD6
- removed net RD7: U1.PMD15/CN16/RD7
- removed net RD8: U1.IC1/RTCC/RD8
- removed net RD9: U1.IC2/SS1/RD9
- removed net RE0: LED3.C, U1.PMD0/RE0
- removed net RE1: LED2.C, U1.PMD1/RE1
- removed net RE2: LED1.C, U1.PMD2/RE2
- removed net RE3: U1.PMD3/RE3, USB.C
- removed net RE4: U1.PMD4/RE4
- removed net RE6: U1.PMD6/RE6
- removed net RE7: U1.PMD7/RE7
- removed net RE9: U1.INT2/RE9
- removed net RF12: U1.U2CTS/RF12
- removed net RF13: U1.U2RTS/BCLK2/RF13
- removed net RF2: U1.U1RX/RF2
- removed net RF4: U1.PMA9/U2RX/CN17/RF4
- removed net RF5: U1.PMA8/U2TX/CN18/RF5
- removed net RF8: U1.U1TX/RF8
- removed net RG0: U1.PMD8/RG0
- removed net RG1: U1.PMD9/RG1
- removed net RG15: U1.RG15
- removed net RG9: U1.PMA2/SS2/CN11/RG9
- removed net SD_CD: U$3.WP, U1.TRD1/RG12
- removed net SD_CK: U$3.SCK, U1.PMA5/SCK2/CN8/RG6
- removed net SD_CS: R16.2, U$3.CS, U1.TRD2/RG14
- removed net SD_DI: U$3.DI, U1.PMA3/SDO2/CN10/RG8
- removed net SD_DO: U$3.DO, U1.PMA4/SDI2/CN9/RG7
- removed net SD_WP: U$3.CD, U1.PMD5/RE5, U1.TRD0/RG13
- removed net USBID: R2.1, U$21.ID, U1.USBID/RF3
- removed net VBUS: U$21.VBUS, U1.VBUS
- removed net VPP: JP1.1, R4.1, U1.MCLR
- removed net WF_CK: R10.1, U$1.SCK, U1.IC3/SCKI/PMCS2/PMA15/RD10
- removed net WF_CS: U$1.CS, U1.SDA2/RA3
- removed net WF_DI: R9.1, U$1.SDI, U1.SDO1/OC1/INT0/RD0
- removed net WF_DO: U$1.SDO, U1.SDI1/T5CK/RC4
- removed net WF_HIBERNATE: U$1.HIBERNATE, U1.PMD10/RF1
- removed net WF_INT: R11.1, U$1.INT, U1.INT1/RE8
- removed net WF_RESET: R7.1, U$1.RESET, U1.PMD11/RF0
- removed net WF_WP: R6.2, U$1.WP
- net AC_HOT: no longer B1.AC1, J1.PWR
- net GND: no longer B1.-, C1.-, C10.-, C11.1, C12.1, C13.2, C14.2, C2.2, C3.2, C4.2, C5.2, C6.2, C7.2, C8.2, C9.2, JP1.3, PWR.C, R6.1, U$1.GND@1, U$1.GND@10, U$1.GND@18, U$1.GND@19, U$1.GND@25, U$1.GND@28, U$1.GND@30, U$1.GND@36, U$21.GND, U$21.MTN1, U$21.MTN2, U$21.MTN3, U$21.MTN4, U$3.GND, U$3.GND1, U$3.SHIELD, U1.AVSS, U1.VSS1, U1.VSS2, U1.VSS3, U1.VSS4, U1.VSS6, U2.GND
Other:
- note removed: "Do Not Populate"
- note removed: "For now WP is held"
- note removed: "ICSP/Debug/IO"
- note removed: "RTC Crystal"
- note removed: "SD CARD"
- note removed: "WI-FI MODULE"
- note removed: "low and not conn."
- note removed: "to the PIC"
- moved on the sheet: OK1, OK10, OK11, OK12, OK13, OK14, OK15, OK16, OK2, OK3, OK4, OK5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

Commit message: First draft of valve board
Parts:
- removed OK11, OK12, OK13, OK14, OK3, OK4, OK5, OK6: MOC3032S, lizardworx:MOC3032S
- removed R26, R27, R28, R29, R30, R31, R32, R33: 330, SparkFun-Passives:RESISTOR0603-RES
- removed R42, R43, R44, R45, R46, R47, R48, R49: 33, SparkFun-Passives:RESISTOR0603-RES
- removed T11, T12, T13, T14, T3, T4, T5, T6: LF-TRIACSOT223, lizardworx:LF-TRIACSOT223
- added JP1: (no value), SparkFun-Connectors:M08LOCK_LONGPADS
Connections:
- removed net CNTRL_10: R27.2
- removed net CNTRL_11: R28.2
- removed net CNTRL_12: R29.2
- removed net CNTRL_13: R30.2
- removed net CNTRL_14: R31.2
- removed net CNTRL_15: R32.2
- removed net CNTRL_16: R33.2
- removed net CNTRL_9: R26.2
- removed net N$17: OK3.A, R26.1
- removed net N$18: OK3.A2, R42.2
- removed net N$21: OK3.A1, T3.G
- removed net N$26: OK4.A, R27.1
- removed net N$27: OK4.A2, R43.2
- removed net N$29: OK4.A1, T4.G
- removed net N$32: OK5.A, R28.1
- removed net N$33: OK5.A2, R44.2
- removed net N$36: OK5.A1, T5.G
- removed net N$39: OK6.A, R29.1
- removed net N$40: OK6.A2, R45.2
- removed net N$42: OK6.A1, T6.G
- removed net N$53: OK11.A, R30.1
- removed net N$57: OK11.A2, R46.2
- removed net N$58: OK11.A1, T11.G
- removed net N$61: OK12.A, R31.1
- removed net N$62: OK12.A2, R47.2
- removed net N$63: OK12.A1, T12.G
- removed net N$66: OK13.A, R32.1
- removed net N$67: OK13.A2, R48.2
- removed net N$68: OK13.A1, T13.G
- removed net N$71: OK14.A, R33.1
- removed net N$72: OK14.A2, R49.2
- removed net N$73: OK14.A1, T14.G
- removed net STATION_10: T4.A1
- removed net STATION_11: T5.A1
- removed net STATION_12: T6.A1
- removed net STATION_13: T11.A1
- removed net STATION_14: T12.A1
- removed net STATION_15: T13.A1
- removed net STATION_16: T14.A1
- removed net STATION_9: T3.A1
- net AC_HOT: no longer R42.1, R43.1, R44.1, R45.1, R46.1, R47.1, R48.1, R49.1, T11.A2, T12.A2, T13.A2, T14.A2, T3.A2, T4.A2, T5.A2, T6.A2
- net CNTRL_1: now also JP1.8
- net CNTRL_2: now also JP1.7
- net CNTRL_3: now also JP1.6
- net CNTRL_4: now also JP1.5
- net CNTRL_5: now also JP1.4
- net CNTRL_6: now also JP1.3
- net CNTRL_7: now also JP1.2
- net CNTRL_8: now also JP1.1
- net GND: no longer OK11.C, OK12.C, OK13.C, OK14.C, OK3.C, OK4.C, OK5.C, OK6.C
