File: hardware/schematic/PIC_WIFI_DEV.sch (EAGLE design)
At the start: 58 parts, among them J5 POWER_JACKPTH, Q1 8MHz, Q2 32.768KHz, U1 PIC32MX460F512L TQFP100, U4 RECOM_X.X_REG78XX

Commit message: Added fuse holder to lib.  Swapped 10k res for 2 4.7K in dev board.  Added fuse to waterworx.sch
Parts:
- added R20: 4.7K, SparkFun:RESISTOR0402
- R9: value 10K -> 4.7K
Connections:
- new net N$6: R20.1, R9.2
- net 3.3V: now also R20.2; no longer R9.2
Other:
- note added: "Need to supply 7.6 to 15V"
- note removed: "Need to supply 7.6 to 42V"
Changed lines of the file:
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@@
 <part name="P+3" library="SparkFun02-20-08" deviceset="3.3V" device=""/>
 <part name="P+15" library="SparkFun02-20-08" deviceset="3.3V" device=""/>
-<part name="R9" library="SparkFun" deviceset="RESISTOR" device="0402" value="10K"/>
+<part name="R9" library="SparkFun" deviceset="RESISTOR" device="0402" value="4.7K"/>
 <part name="R3" library="SparkFun" deviceset="RESISTOR" device="0402" value="4.7K"/>
 <part name="R5" library="SparkFun" deviceset="RESISTOR" device="0402" value="4.7K"/>
@@
 <part name="JP5" library="SparkFun-Connectors" deviceset="M15" device=""/>
 <part name="JP3" library="SparkFun-Connectors" deviceset="M16" device="PTH"/>
+<part name="R20" library="SparkFun" deviceset="RESISTOR" device="0402" value="4.7K"/>
 </parts>
 <sheets>
@@
 <wire x1="137.16" y1="238.76" x2="93.98" y2="238.76" width="0.1524" layer="98"/>
 <text x="91.44" y="149.86" size="1.778" layer="98" rot="R90">Power ON LED</text>
-<text x="8.636" y="190.246" size="1.778" layer="98">Need to supply 7.6 to 42V</text>
+<text x="8.636" y="190.246" size="1.778" layer="98">Need to supply 7.6 to 15V</text>
 <text x="15.24" y="182.88" size="1.778" layer="98">Diode has .5V voltage drop</text>
 <text x="15.24" y="208.28" size="1.778" layer="98">Do Not Populate</text>
@@
 <instance part="GND2" gate="1" x="76.2" y="208.28"/>
 <instance part="P+3" gate="G$1" x="289.56" y="111.76" rot="R270"/>
-<instance part="P+15" gate="G$1" x="302.26" y="101.6" rot="R270"/>
+<instance part="P+15" gate="G$1" x="314.96" y="101.6" rot="R270"/>
 <instance part="R9" gate="G$1" x="294.64" y="101.6"/>
 <instance part="R3" gate="G$1" x="355.6" y="106.68" rot="R270"/>
@@
 <instance part="JP5" gate="G$1" x="248.92" y="53.34" rot="R270"/>
 <instance part="JP3" gate="G$1" x="251.46" y="208.28" rot="R90"/>
+<instance part="R20" gate="G$1" x="309.88" y="101.6"/>
 </instances>
 <busses>
@@
 </segment>
 <segment>
-<wire x1="299.72" y1="101.6" x2="302.26" y2="101.6" width="0.1524" layer="91"/>
-<pinref part="R9" gate="G$1" pin="2"/>
-<pinref part="P+15" gate="G$1" pin="3.3V"/>
-</segment>
-<segment>
 <wire x1="264.16" y1="43.18" x2="264.16" y2="30.48" width="0.1524" layer="91"/>
 <pinref part="P+5" gate="G$1" pin="3.3V"/>
@@
 <pinref part="P+18" gate="G$1" pin="3.3V"/>
 <wire x1="355.6" y1="195.58" x2="355.6" y2="193.04" width="0.1524" layer="91"/>
+</segment>
+<segment>
+<pinref part="P+15" gate="G$1" pin="3.3V"/>
+<pinref part="R20" gate="G$1" pin="2"/>
 </segment>
 </net>
@@
 </segment>
 </net>
+<net name="N$6" class="0">
+<segment>
+<pinref part="R9" gate="G$1" pin="2"/>
+<pinref part="R20" gate="G$1" pin="1"/>
+<wire x1="304.8" y1="101.6" x2="299.72" y2="101.6" width="0.1524" layer="91"/>
+</segment>
+</net>
